File: Hardware/Qwiic-Bluetooth-HC1X.sch (EAGLE design)
At the start: 31 parts, among them J1 ISP, J2 Qwiic-L, J3 Qwiic-R, J4 I2C, J5 PIO, U1 ATTiny85-Arduino, U2 HM-17

Commit message: Adding decoupling, fixing silk.
Parts:
- added C3: 4.7uF, SparkFun-Capacitors:4.7UF0603
- added C4: 10uF, SparkFun-Capacitors:10UF-0603-6.3V-20%
- JP3: value JUMPER-SMT_3_2-NC_TRACE_SILK -> I2C; device SparkFun-Jumpers:JUMPER-SMT_3_2-NC_TRACE_SILK -> SparkFun-Jumpers:JUMPER-SMT_3_2-NC_TRACE_NO-SILK
- JP4: device SparkFun-Jumpers:JUMPER-SMT_2_NC_TRACE_SILK -> SparkFun-Jumpers:JUMPER-SMT_2_NC_TRACE_NO-SILK
Connections:
- net PIO1 renamed PIO1/LED
- net 3.3V: now also C3.1, C4.1
- net GND: now also C3.2, C4.2
Other:
- moved on the sheet: JP1, S1, U2

Commit message: Fixing HM-17 pinout, and revising layout to x02
Parts:
- C3: device SparkFun-Capacitors:4.7UF0603 -> SparkFun-Capacitors:4.7UF-0603-6.3V-(10%)
- LOGO2: value SPARKX-LOGO3 -> SPARKX-LOGO4; device SparkX:SPARKX-LOGO3 -> SparkX:SPARKX-LOGO4
Other:
- note added: "X02"
- note removed: "X01"
Changed lines of the file:
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@@
 <part name="LOGO3" library="SparkX" deviceset="SPARKX-LOGO" device="4"/>
 <part name="LOGO1" library="SparkFun-Aesthetics" deviceset="OSHW-LOGO" device="MINI"/>
-<part name="LOGO2" library="SparkX" deviceset="SPARKX-LOGO" device="3" value="SPARKX-LOGO3"/>
+<part name="LOGO2" library="SparkX" deviceset="SPARKX-LOGO" device="4" value="SPARKX-LOGO4"/>
 <part name="JP8" library="SparkFun-Aesthetics" deviceset="FIDUCIAL" device="UFIDUCIAL"/>
 <part name="JP6" library="SparkFun-Aesthetics" deviceset="FIDUCIAL" device="UFIDUCIAL"/>
@@
 <part name="GND2" library="SparkFun-PowerSymbols" deviceset="GND" device=""/>
 <part name="SUPPLY3" library="SparkFun-PowerSymbols" deviceset="3.3V" device=""/>
-<part name="C3" library="SparkFun-Capacitors" deviceset="4.7UF" device="0603" value="4.7uF"/>
+<part name="C3" library="SparkFun-Capacitors" deviceset="4.7UF" device="-0603-6.3V-(10%)" value="4.7uF"/>
 <part name="SUPPLY12" library="SparkFun-PowerSymbols" deviceset="3.3V" device=""/>
 <part name="GND13" library="SparkFun-PowerSymbols" deviceset="GND" device=""/>
@@
 <text x="2.54" y="182.88" size="3.81" layer="97" ratio="15" align="top-left">ATtiny85</text>
 <text x="165.354" y="11.43" size="2.54" layer="94">Jim Lindblom</text>
-<text x="237.744" y="7.366" size="2.54" layer="94">X01</text>
+<text x="237.744" y="7.366" size="2.54" layer="94">X02</text>
 <text x="204.343" y="136.271" size="1.778" layer="97" rot="R90">Power</text>
 <text x="9.398" y="40.64" size="1.778" layer="97" align="top-left">Key-select provides KEY button support
